File: 3D modeling/회로도.kicad_sch/회로도.kicad_sch.kicad_pcb (KiCad board)
At the start: 2 copper layers, 94 x 91.5 mm, 6 parts, among them J1 PinHeader_1x15_P2.54mm_Vertic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, J2 PinHeader_1x15_P2.54mm_Vertic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, J3 PinHeader_1x08_P2.54mm_Vertic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, J4 PinHeader_1x05_P2.54mm_Vertic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, J5 PinHeader_1x05_P2.54mm_Vertic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, J6 PinHeader_1x05_P2.54mm_Vertic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

Commit message: 배선도 추가:
Connections:
- J1 pad 1: (no net) -> 3V3
- J1 pad 10: (no net) -> GPIO26
- J1 pad 11: (no net) -> GPIO27
- J1 pad 12: (no net) -> GPIO14
- J1 pad 13: (no net) -> GPIO12
- J1 pad 14: (no net) -> GPIO13
- J1 pad 15: (no net) -> GND
- J1 pad 2: (no net) -> ESP_EN
- J1 pad 3: (no net) -> GPIO36
- J1 pad 4: (no net) -> GPIO39
- J1 pad 5: (no net) -> GPIO34
- J1 pad 6: (no net) -> GPIO35
- J1 pad 7: (no net) -> GPIO32
- J1 pad 8: (no net) -> GPIO33
- J1 pad 9: (no net) -> GPIO25
- J2 pad 1: (no net) -> 5V
- J2 pad 10: (no net) -> GPIO19
- J2 pad 11: (no net) -> I2C_SDA
- J2 pad 12: (no net) -> GPIO3
- J2 pad 13: (no net) -> GPIO1
- J2 pad 14: (no net) -> I2C_SCL
- J2 pad 15: (no net) -> GPIO23
- J2 pad 2: (no net) -> GND
- J2 pad 3: (no net) -> GPIO15
- J2 pad 4: (no net) -> GPIO2
- J2 pad 5: (no net) -> GPIO4
- J2 pad 6: (no net) -> GPS_TX
- J2 pad 7: (no net) -> GPS_RX
- J2 pad 8: (no net) -> GPIO5
- J2 pad 9: (no net) -> GPIO18
- J3 pad 1: (no net) -> 3V3
- J3 pad 2: (no net) -> GND
- J3 pad 3: (no net) -> I2C_SCL
- J3 pad 4: (no net) -> I2C_SDA
- J3 pad 5: (no net) -> GY_XDA
- J3 pad 6: (no net) -> GY_XCL
- J3 pad 7: (no net) -> GY_AD0
- J3 pad 8: (no net) -> GY_INT
- J4 pad 1: (no net) -> 3V3
- J4 pad 2: (no net) -> GND
- J4 pad 3: (no net) -> I2C_SCL
- J4 pad 4: (no net) -> I2C_SDA
- J4 pad 5: (no net) -> SHT_ALR
- J5 pad 1: (no net) -> 5V
- J5 pad 2: (no net) -> GPS_RX
- J5 pad 3: (no net) -> GPS_TX
- J5 pad 4: (no net) -> GND
- J5 pad 5: (no net) -> GPS_PPS
- J6 pad 1: (no net) -> 3V3
- J6 pad 2: (no net) -> GND
- J6 pad 3: (no net) -> I2C_SCL
- J6 pad 4: (no net) -> I2C_SDA
- J6 pad 5: (no net) -> BH_ADD
Routing:
- net GND: track 0.00 -> 162.6 mm
- net I2C_SCL: track 0.00 -> 134.6 mm, vias 0 -> 1
- net 3V3: track 0.00 -> 101.0 mm
- net I2C_SDA: track 0.00 -> 78.7 mm
- net 5V: track 0.00 -> 39.9 mm
- net GPS_TX: track 0.00 -> 30.5 mm
- net GPS_RX: track 0.00 -> 30.5 mm
Other:
- board size 94 x 91.5 mm -> 94 x 71 mm
