File: 3D modeling/회로도_stack/회로도_stack.kicad_pcb (KiCad board)
At the start: 2 copper layers, 153.4 x 55.9 mm, 5 parts, among them J1 PinHeader_1x22_P2.54mm_Vertic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, J2 PinHeader_1x22_P2.54mm_Vertic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, J4 PinHeader_1x05_P2.54mm_Vertic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, J5 PinHeader_1x05_P2.54mm_Vertic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, J6 PinHeader_1x05_P2.54mm_Vertic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

Commit message: 배선도 추가:
Connections:
- J1 pad 1: (no net) -> 3V3
- J1 pad 10: (no net) -> IO18
- J1 pad 11: (no net) -> I2C_SDA
- J1 pad 12: (no net) -> IO19
- J1 pad 13: (no net) -> IO20
- J1 pad 14: (no net) -> IO3
- J1 pad 15: (no net) -> IO46
- J1 pad 16: (no net) -> I2C_SCL
- J1 pad 17: (no net) -> IO10
- J1 pad 18: (no net) -> IO11
- J1 pad 19: (no net) -> IO12
- J1 pad 2: (no net) -> EN
- J1 pad 20: (no net) -> IO13
- J1 pad 21: (no net) -> IO14
- J1 pad 22: (no net) -> GND
- J1 pad 3: (no net) -> IO4
- J1 pad 4: (no net) -> IO5
- J1 pad 5: (no net) -> IO6
- J1 pad 6: (no net) -> IO7
- J1 pad 7: (no net) -> IO15
- J1 pad 8: (no net) -> GPS_RX
- J1 pad 9: (no net) -> GPS_TX
- J2 pad 1: (no net) -> GND
- J2 pad 10: (no net) -> IO38
- J2 pad 11: (no net) -> IO39
- J2 pad 12: (no net) -> IO40
- J2 pad 13: (no net) -> IO41
- J2 pad 14: (no net) -> IO42
- J2 pad 15: (no net) -> IO44
- J2 pad 16: (no net) -> IO43
- J2 pad 17: (no net) -> IO2
- J2 pad 18: (no net) -> IO1
- J2 pad 19: (no net) -> IO26
- J2 pad 2: (no net) -> IO21
- J2 pad 20: (no net) -> IO25
- J2 pad 21: (no net) -> 5V
- J2 pad 22: (no net) -> GND
- J2 pad 3: (no net) -> IO47
- J2 pad 4: (no net) -> IO48
- J2 pad 5: (no net) -> IO45
- J2 pad 6: (no net) -> IO0
- J2 pad 7: (no net) -> IO35
- J2 pad 8: (no net) -> IO36
- J2 pad 9: (no net) -> IO37
- J4 pad 1: (no net) -> 3V3
- J4 pad 2: (no net) -> GND
- J4 pad 3: (no net) -> I2C_SCL
- J4 pad 4: (no net) -> I2C_SDA
- J4 pad 5: (no net) -> SHT_ALR
- J5 pad 1: (no net) -> 5V_BOT
- J5 pad 2: (no net) -> GPS_RX_BOT
- J5 pad 3: (no net) -> GPS_TX_BOT
- J5 pad 4: (no net) -> GND_BOT
- J5 pad 5: (no net) -> GPS_PPS
- J6 pad 1: (no net) -> 3V3_BOT
- J6 pad 2: (no net) -> GND_BOT
- J6 pad 3: (no net) -> I2C_SCL_BOT
- J6 pad 4: (no net) -> I2C_SDA_BOT
- J6 pad 5: (no net) -> BH_ADD
Routing:
- net GND: track 0.00 -> 97.6 mm
- net I2C_SCL: track 0.00 -> 83.6 mm
- net I2C_SDA: track 0.00 -> 76.8 mm
- net 3V3: track 0.00 -> 36.6 mm
- net GND_BOT: track 0.00 -> 9.72 mm
